File: Artemis Charger Mod PCB.brd (EAGLE design)
At the start: 100 x 80 mm, 45 parts, among them J2 MOLEX_CLICKMATE-4-VERTICAL, U1 CSD17506Q5A, U10 TPS562219, U2 FAN3214, U3 MAX5812, U4 FAN3214, U5 CSD17506Q5A, U6 CSD17506Q5A, U7 CSD17506Q5A, U8 MAX5812, U9 TPS562219

Commit message: Almost Done
Parts:
- added C10, C11: 10uF, adafruit:C0805
- added C18: 8200pF, adafruit:C0805
- added C21, C9: 0.1uF, adafruit:C0805
- added C22, C23, C24: 22uF, adafruit:C0805
- added J1, J3: MOLEX_CLICKMATE-4-VERTICAL, FormE:MOLEX-CLIKMATE-4-VERTICAL-HEADER
- added J4, J5: MOLEX_CLICKMATE-2-VERTICAL, FormE:MOLEX-CLIKMATE-2-VERTICAL-HEADER
- added L3: 4.7uH, FormE:SRP6540
- added LED2: GREEN, FormE:CHIPLED_0805
- added R10: 1K, adafruit:R0805
- added R11, R8, R9: 10K, adafruit:R0805
- added R7: 54.9k, adafruit:R0805
- added U11, U12: ISO7340, FormE:ISO734X
- added U13: TPS562219, FormE:TPS562219
- R1: value 54.9k -> 33.2k
Connections:
- new net N$24: JP1.29, U11.P$4
- new net N$27: JP1.13, U11.P$6
- new net N$29: JP1.15, U11.P$5
- new net N$30: J1.4, U11.P$11
- new net N$31: J1.3, U11.P$12
- new net N$32: J1.2, U11.P$13
- new net N$33: J1.1, U11.P$14
- new net N$34: J3.4, U12.P$3
- new net N$35: J3.3, U12.P$4
- new net N$36: J3.2, U12.P$5
- new net N$37: J3.1, U12.P$6
- new net N$38: JP1.18, U12.P$14
- new net N$39: JP1.16, U12.P$13
- new net N$40: JP1.12, U12.P$12
- new net N$41: JP1.7, U12.P$11
- new net N$42: J4.2, J5.1
- new net N$43: J5.2, JP1.11, R11.2
- new net N$44: R9.2, U13.7
- new net N$45: LED2.C, R10.2
- new net N$5: JP1.31, U11.P$3
- new net SS_5V2: C18.1, U13.5
- new net SW_5V2: C21.2, L3.P$1, U13.2
- new net VBST_5V2: C21.1, U13.8
- new net VFB_5V2: R7.1, R8.2, U13.6
- net +5V: now also U11.P$16, U12.P$1
- net +5V/1: now also C22.1, C23.1, C24.1, J4.1, L3.P$2, LED2.A, R7.2, U11.P$1, U12.P$16
- net GND: now also U11.P$15, U11.P$9, U12.P$2, U12.P$8
- net GND1: now also C10.2, C11.2, C18.2, C22.2, C23.2, C24.2, C9.2, R10.1, R11.1, R8.1, U11.P$2, U11.P$8, U12.P$15, U12.P$9, U13.1
- net VDD: now also C10.1, C11.1, C9.1, R9.1, U13.3
Routing:
- net GND1: track 167.9 -> 218.3 mm, vias 11 -> 13
- net N$44: track 0.00 -> 16.7 mm
- net SW_5V2: track 0.00 -> 10.2 mm
- net VDD: track 137.0 -> 147.1 mm
- net +5V/1: track 126.0 -> 136.1 mm
- net VBST_5V2: track 0.00 -> 6.93 mm
