File: Artemis Charger Mod PCB.2.sch (EAGLE design)
At the start: 159 parts, among them J1 MOLEX_CLICKMATE-2-VERTICAL, J2 MOLEX_CLICKMATE-4-VERTICAL, J3 MOLEX_CLICKMATE-2-VERTICAL, J4 MOLEX_CLICKMATE-2-VERTICAL, J5 MOLEX_CLICKMATE-2-VERTICAL, J6 MOLEX_CLICKMATE-2-VERTICAL, Q10 BSS138, Q11 BSS138, Q8 BSS138, Q9 BSS138, U10 TPS562219, U11 ISO7340, U12 ISO7340, U13 TPS562219, U14 MCP2515-TSSOP, U15 MCP2562, U17 CD4050BD, U18 CD4043B, U19 SN74LVC08ASOIC, U20 SN74LVC32ASOIC, U22 LTC1155, U23 CSD17506Q5A, U26 CSD17506Q5A, U27 LTC1155, U28 CSD17506Q5A, U29 LTC1155, U3 MAX5812, U30 CSD17506Q5A, U32 CSD17506Q5A, U34 CSD17506Q5A, U49 TL7712A-SOIC, U8 MAX5812, U9 TPS562219

Commit message: Added STENCIL
Parts:
- H2, H3: PARTNO (none) -> 5025840870
- H4: PARTNO (none) -> 5025841170
- J1, J3, J4, J5, J6: PARTNO (none) -> 5025840270
- J2: PARTNO (none) -> 5040500491
- U3, U8: value MAX5812 -> MAX5812LEUT+TCT-ND
Changed lines of the file:
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@@
 <attribute name="PARTNO" value="ISO1541DR"/>
 </part>
-<part name="U3" library="FormE" deviceset="MAX5812" device="M" value="MAX5812">
+<part name="U3" library="FormE" deviceset="MAX5812" device="M" value="MAX5812LEUT+TCT-ND">
 <attribute name="PARTNO" value="MAX5812LEUT+T"/>
 </part>
@@
 <part name="GND22" library="supply1" deviceset="GND" device=""/>
 <part name="P+21" library="supply1" deviceset="+5V" device=""/>
-<part name="U8" library="FormE" deviceset="MAX5812" device="M" value="MAX5812">
+<part name="U8" library="FormE" deviceset="MAX5812" device="M" value="MAX5812LEUT+TCT-ND">
 <attribute name="PARTNO" value="MAX5812LEUT+T"/>
 </part>
@@
 <part name="SUPPLY6" library="supply2" deviceset="GND1" device=""/>
 <part name="SUPPLY5" library="supply2" deviceset="GND1" device=""/>
-<part name="H2" library="FormE" deviceset="MOLEX_CLIKMATE-8-VERTICAL" device=""/>
-<part name="J2" library="FormE" deviceset="MOLEX_CLICKMATE-4-VERTICAL" device=""/>
+<part name="H2" library="FormE" deviceset="MOLEX_CLIKMATE-8-VERTICAL" device="">
+<attribute name="PARTNO" value="5025840870"/>
+</part>
+<part name="J2" library="FormE" deviceset="MOLEX_CLICKMATE-4-VERTICAL" device="">
+<attribute name="PARTNO" value="5040500491"/>
+</part>
 <part name="SUPPLY22" library="supply2" deviceset="GND1" device=""/>
 <part name="SUPPLY7" library="supply1" deviceset="+3V3" device=""/>
@@
 <part name="SUPPLY35" library="supply2" deviceset="+5V/1" device=""/>
 <part name="SUPPLY36" library="supply2" deviceset="VDD" device=""/>
-<part name="H3" library="FormE" deviceset="MOLEX_CLIKMATE-8-VERTICAL" device=""/>
+<part name="H3" library="FormE" deviceset="MOLEX_CLIKMATE-8-VERTICAL" device="">
+<attribute name="PARTNO" value="5025840870"/>
+</part>
 <part name="U14" library="FormE" deviceset="MCP2515" device="-TSSOP">
 <attribute name="MF" value=""/>
@@
 <attribute name="PARTNO" value="ERJ-6ENF1200V"/>
 </part>
-<part name="H4" library="FormE" deviceset="MOLEX_CLICKMATE-11-VERTICAL" device="-VERTICAL"/>
+<part name="H4" library="FormE" deviceset="MOLEX_CLICKMATE-11-VERTICAL" device="-VERTICAL">
+<attribute name="PARTNO" value="5025841170"/>
+</part>
 <part name="SUPPLY38" library="supply1" deviceset="+3V3" device=""/>
 <part name="SUPPLY37" library="supply2" deviceset="+5V/1" device=""/>
@@
 <part name="SUPPLY15" library="supply2" deviceset="GND1" device=""/>
 <part name="SUPPLY14" library="supply2" deviceset="GND1" device=""/>
-<part name="J1" library="FormE" deviceset="MOLEX_CLICKMATE-2-VERTICAL" device=""/>
-<part name="J3" library="FormE" deviceset="MOLEX_CLICKMATE-2-VERTICAL" device=""/>
-<part name="J4" library="FormE" deviceset="MOLEX_CLICKMATE-2-VERTICAL" device=""/>
-<part name="J5" library="FormE" deviceset="MOLEX_CLICKMATE-2-VERTICAL" device=""/>
+<part name="J1" library="FormE" deviceset="MOLEX_CLICKMATE-2-VERTICAL" device="">
+<attribute name="PARTNO" value="5025840270"/>
+</part>
+<part name="J3" library="FormE" deviceset="MOLEX_CLICKMATE-2-VERTICAL" device="">
+<attribute name="PARTNO" value="5025840270"/>
+</part>
+<part name="J4" library="FormE" deviceset="MOLEX_CLICKMATE-2-VERTICAL" device="">
+<attribute name="PARTNO" value="5025840270"/>
+</part>
+<part name="J5" library="FormE" deviceset="MOLEX_CLICKMATE-2-VERTICAL" device="">
+<attribute name="PARTNO" value="5025840270"/>
+</part>
 <part name="SUPPLY16" library="supply2" deviceset="GND1" device=""/>
 <part name="SUPPLY17" library="supply2" deviceset="GND1" device=""/>
@@
 </part>
 <part name="SUPPLY58" library="supply1" deviceset="+3V3" device=""/>
-<part name="J6" library="FormE" deviceset="MOLEX_CLICKMATE-2-VERTICAL" device=""/>
+<part name="J6" library="FormE" deviceset="MOLEX_CLICKMATE-2-VERTICAL" device="">
+<attribute name="PARTNO" value="5025840270"/>
+</part>
 </parts>
 <sheets>
@@
 <instance part="SUPPLY6" gate="G$1" x="215.9" y="109.22"/>
 <instance part="SUPPLY5" gate="G$1" x="-5.08" y="124.46"/>
-<instance part="H2" gate="G$1" x="307.34" y="15.24" rot="R270"/>
-<instance part="J2" gate="G$1" x="-25.4" y="172.72" rot="R90"/>
+<instance part="H2" gate="G$1" x="307.34" y="15.24" rot="R270">
+<attribute name="PARTNO" x="307.34" y="15.24" size="1.778" layer="96" display="off"/>
+</instance>
+<instance part="J2" gate="G$1" x="-25.4" y="172.72" rot="R90">
+<attribute name="PARTNO" x="-25.4" y="172.72" size="1.778" layer="96" display="off"/>
+</instance>
 <instance part="SUPPLY22" gate="G$1" x="-33.02" y="162.56" rot="R270"/>
 <instance part="SUPPLY7" gate="G$1" x="180.34" y="152.4"/>
@@
 <instance part="SUPPLY35" gate="G$1" x="215.9" y="330.2"/>
 <instance part="SUPPLY36" gate="G$1" x="-35.56" y="332.74"/>
-<instance part="H3" gate="G$1" x="386.08" y="93.98"/>
+<instance part="H3" gate="G$1" x="386.08" y="93.98">
+<attribute name="PARTNO" x="386.08" y="93.98" size="1.778" layer="96" display="off"/>
+</instance>
 <instance part="U14" gate="G$1" x="510.54" y="157.48">
 <attribute name="PARTNO" x="510.54" y="157.48" size="1.778" layer="96" display="off"/>
@@
 <attribute name="MPN" x="535.94" y="195.58" size="1.778" layer="96" display="off"/>
 </instance>
-<instance part="H4" gate="G$1" x="368.3" y="251.46" rot="R180"/>
+<instance part="H4" gate="G$1" x="368.3" y="251.46" rot="R180">
+<attribute name="PARTNO" x="368.3" y="251.46" size="1.778" layer="96" display="off"/>
+</instance>
 <instance part="SUPPLY38" gate="G$1" x="383.54" y="261.62" rot="R270"/>
 <instance part="SUPPLY37" gate="G$1" x="596.9" y="203.2"/>
@@
 <instance part="SUPPLY15" gate="G$1" x="492.76" y="452.12"/>
 <instance part="SUPPLY14" gate="G$1" x="566.42" y="459.74"/>
-<instance part="J1" gate="G$1" x="904.24" y="391.16"/>
-<instance part="J3" gate="G$1" x="904.24" y="381"/>
-<instance part="J4" gate="G$1" x="904.24" y="350.52"/>
-<instance part="J5" gate="G$1" x="904.24" y="340.36"/>
+<instance part="J1" gate="G$1" x="904.24" y="391.16">
+<attribute name="PARTNO" x="904.24" y="391.16" size="1.778" layer="96" display="off"/>
+</instance>
+<instance part="J3" gate="G$1" x="904.24" y="381">
+<attribute name="PARTNO" x="904.24" y="381" size="1.778" layer="96" display="off"/>
+</instance>
+<instance part="J4" gate="G$1" x="904.24" y="350.52">
+<attribute name="PARTNO" x="904.24" y="350.52" size="1.778" layer="96" display="off"/>
+</instance>
+<instance part="J5" gate="G$1" x="904.24" y="340.36">
+<attribute name="PARTNO" x="904.24" y="340.36" size="1.778" layer="96" display="off"/>
+</instance>
 <instance part="SUPPLY16" gate="G$1" x="891.54" y="373.38"/>
 <instance part="SUPPLY17" gate="G$1" x="891.54" y="304.8"/>
@@
 </instance>
 <instance part="SUPPLY58" gate="G$1" x="546.1" y="177.8"/>
-<instance part="J6" gate="G$1" x="904.24" y="325.12"/>
+<instance part="J6" gate="G$1" x="904.24" y="325.12">
+<attribute name="PARTNO" x="904.24" y="325.12" size="1.778" layer="96" display="off"/>
+</instance>
 </instances>
 <busses>

Commit message: Cleaned up sch
Other:
- note added: "Charger Board"
- note added: "Connect to PI"
- note added: "DAC's"
- note added: "Isolated Charger Side"
- note added: "Level Shifters"
- note added: "MISC. Connectors"
- note added: "Outputs connect to PI"
- note added: "Power in from power brick 15V=VDD"
- note added: "Rassberry PI Connector"
- note added: "These 4 conectors to contactors in charger enclosure"
- note added: "Voltage Regulators"
- note added: "Voltage Supervisor"
- note removed: "<-- These 4 conectors to contactors in charger enclosure"
- note removed: "<-- To contactor in Acumulator"
- note removed: "Goes to IO Pannle, Connect to others"
- note removed: "Power in from power brick, 15V=VDD"
- note removed: "To Voltage supervisor"
- note removed: "pull +12V to 15V PI side instead"
- moved on the sheet: C1, C10, C11, C12, C13, C14, C15, C16, C17, C18, C19, C2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
